File: pcb/MiSTer_LLOAD_DIY_Edition.brd (EAGLE design)
At the start: 100 x 80 mm, 16 parts, among them IC3 REG1117, K1 692121030100

Commit message: Removed alternate VCC (3.3v) from DB15 pin 10. This will not make it directly compatible with supergun input, but at least no harm will be done in case someone inadvertently uses a supergun with it. Neo Geo and Neo Geo CD are still welcome in both revisions.
Connections:
- net 3V3: no longer X1.10, X2.10
Routing:
- net 3V3: track 168.4 -> 112.1 mm
- net D7: track 59.2 -> 80.9 mm, vias 1 -> 0
- net P2_F5: track 66.1 -> 54.4 mm, vias 0 -> 1
- net P2_B7: track 72.5 -> 75.0 mm
- net P2_VCC: track 57.3 -> 59.1 mm
- net C6: track 39.2 -> 41.0 mm
- net P2_B4: track 60.6 -> 58.9 mm
- net P2_E6: track 65.0 -> 66.5 mm
- net C7: track 79.1 -> 77.6 mm
- net P2_C7: track 68.8 -> 67.8 mm
- net P2_B5: track 61.8 -> 61.2 mm
- net B5: track 72.8 -> 73.3 mm
- net P2_F4: vias 0 -> 1
- net P2_F1: vias 0 -> 1
Other:
- board text added: "LLOAD - Low Latency Open Adapter for MiSTer FPGA v1.1"
- board text removed: "LLOAD - Low Latency Open Adapter for MiSTer FPGA v1.0"
